File: gachapaw/tof_mount/tof_mount.kicad_pcb (KiCad board)
At the start: 2 copper layers, 40.1 x 45.9 mm, 38 parts, among them J1 PHONE_CHARGER, J3 IN, Q1 AO3400A, Q2 BSS138, U1 VL53L1CXV0FY1, U2 ME6211C28M5, U3 CH32V003F4P6, U4 XL1509-5.0

Commit message: very basic software
Parts:
- removed REF**: boykisser_10mm, pawprint_kicad_art:boykisser_10mm
- removed REF**: logo_designed_at, pawprint_kicad_art:logo_designed_at
- added D5: LED, Resistor_SMD:R_0603_1608Metric, F.Cu at (176.4, 113.8)
- added R11: 10k, Resistor_SMD:R_0402_1005Metric, F.Cu at (168.7, 95.7)
- added R12: 10k, Resistor_SMD:R_0402_1005Metric, F.Cu at (176.4, 95.7)
- added R13: 10k, Resistor_SMD:R_0402_1005Metric, F.Cu at (184.1, 99.7)
- added R14: 330, Resistor_SMD:R_0402_1005Metric, F.Cu at (176.4, 111.1)
- added SW1: BT1, Button_Switch_SMD:SW_SPST_EVPBF, F.Cu at (180.2, 92.2)
- added SW2: BT2, Button_Switch_SMD:SW_SPST_EVPBF, F.Cu at (172.5, 92.2)
- added SW3: RESET, Button_Switch_SMD:SW_SPST_EVPBF, F.Cu at (180.2, 101.9)
- moved C2 0.80 mm to (178.0, 121.4)
- moved R2 0.80 mm to (178.0, 118.4)
Connections:
- J3 pad 7: GND -> /~{RST}
- U3 pad 14: unconnected-(U3-PC4-Pad14) -> /LED
- U3 pad 15: unconnected-(U3-PC5-Pad15) -> /BT1
- U3 pad 16: unconnected-(U3-PC6-Pad16) -> /BT2
Routing:
- net /~{RST}: track 2.67 -> 62.7 mm, vias 0 -> 2
- net +2V8: track 54.2 -> 106.3 mm, vias 3 -> 8
- net /BT2: track 0.00 -> 41.1 mm, vias 0 -> 4
- net /BT1: track 0.00 -> 39.7 mm, vias 0 -> 4
- net /LED: track 0.00 -> 11.9 mm, vias 0 -> 2
- net GND: track 18.6 -> 20.7 mm, vias 11 -> 16
- net +5V: track 64.9 -> 66.7 mm
- net /UART_TX: track 20.1 -> 21.7 mm
- net Net-(D5-A): track 0.00 -> 1.36 mm
- net /UART_RX: track 24.0 -> 25.1 mm
Other:
- board text added: "RST"
- board text added: "SOLENOID"
- board text removed: "SOL"
