File: gachapaw/tof_mount/tof_mount.kicad_sch (KiCad schematic)
At the start: 36 parts, among them J1 PHONE_CHARGER, J3 IN, Q1 AO3400A, Q2 BSS138, U1 VL53L1CXV0FY1, U2 ME6211C28M5, U3 CH32V003F4P6, U4 XL1509-5.0

Commit message: very basic software
Parts:
- added D5: LED, Resistor_SMD:R_0603_1608Metric, symbol Device:LED
- added R11, R12, R13: 10k, Resistor_SMD:R_0402_1005Metric, symbol Device:R
- added R14: 330, Resistor_SMD:R_0402_1005Metric, symbol Device:R
- added SW1: BT1, Button_Switch_SMD:SW_SPST_EVPBF, symbol Switch:SW_SPST
- added SW2: BT2, Button_Switch_SMD:SW_SPST_EVPBF, symbol Switch:SW_SPST
- added SW3: RESET, Button_Switch_SMD:SW_SPST_EVPBF, symbol Switch:SW_SPST
Connections:
- net +2V8: now also R11.1, R12.1, R13.1, R14.1
- net GND: now also SW1.2 (B), SW2.2 (B), SW3.1 (A); no longer J3.7 (Pin_7)
- net ~{RST}: now also J3.7 (Pin_7), R13.2, SW3.2 (B)
- net LED: now reaches U3.14 (PC4)
- net LED: now also D5.1 (K)
- net BT1: now reaches U3.15 (PC5)
- net BT1: now also R12.2, SW1.1 (A)
- net BT2: now reaches U3.16 (PC6)
- net BT2: now also R11.2, SW2.1 (A)
- new net: D5.2 (A), R14.2
- no-connect marks 12 -> 9
Other:
- moved on the sheet: C1, C2, C3, C4, C5, C6, C7, C8, D1, D2, D3, D4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
